File: erc_demo2.kicad_sch (KiCad schematic)
At the start: 11 parts, among them J3 Conn_01x02, J4 Conn_01x04, J5 Conn_01x04

Commit message: feat: kicad9 scheets updated
Parts:
- removed J3: Conn_01x02, symbol Connector_Generic:Conn_01x02
- removed J4, J5: Conn_01x04, symbol Connector_Generic:Conn_01x04
- added J1, J3: Conn_01x04, symbol Connector_Generic:Conn_01x04
- added J2: Conn_01x02, symbol Connector_Generic:Conn_01x02
- R1, R3, R5, R7: value 100k -> 10k
- R2, R4, R6, R8: value 10k -> 100k
Connections:
- net +3V3: now also R1.1, R3.1, R5.1, R7.1, J2.2 (Pin_2); no longer R2.1, R4.1, R6.1, R8.1
- net GND: now also R2.2, R4.2, R6.2, R8.2, J2.1 (Pin_1); no longer R1.2, R3.2, R5.2, R7.2
- new net: J1.1 (Pin_1), J1.4 (Pin_4), J3.1 (Pin_1), J3.4 (Pin_4), R1.2, R2.1, R7.2, R8.1
- new net: J1.2 (Pin_2), J3.2 (Pin_2), R5.2, R6.1
- new net: J1.3 (Pin_3), J3.3 (Pin_3), R3.2, R4.1
