File: erc_demo3.kicad_sch (KiCad schematic)
At the start: 11 parts, among them J3 Conn_01x02, J4 Conn_01x04, J5 Conn_01x04

Commit message: feat: kicad9 scheets updated
Parts:
- renumbered J5 to J4, J3 to J5, J4 to J6, R1 to R10, R4 to R11, R3 to R12, R6 to R13, R5 to R14, R8 to R15, R7 to R16, R2 to R9
Connections:
- net +3V3: no longer J5.2 (Pin_2)
- new net 3V3: J5.2 (Pin_2)
Changed lines of the file:
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@@
+		)
+	)
+	(label "3V3"
+		(at 49.53 26.67 0)
+		(effects
+			(font
+				(size 1.27 1.27)
+			)
+			(justify left bottom)
 		)
 	)
@@
 		)
 	)
+	(label "GND"
+		(at 49.53 29.21 0)
+		(effects
+			(font
+				(size 1.27 1.27)
+			)
+			(justify left bottom)
+		)
+	)
 	(label "Gpo-N33"
 		(at 38.1 67.31 0)
@@
 	)
 	(symbol
-		(lib_id "power:+3V3")
-		(at 49.53 26.67 0)
-		(unit 1)
-		(exclude_from_sim no)
-		(in_bom yes)
-		(on_board yes)
-		(dnp no)
-		(fields_autoplaced yes)
-		(property "Reference" "#PWR1"
-			(at 49.53 30.48 0)
-			(effects
-				(font
-					(size 1.27 1.27)
-				)
-				(hide yes)
-			)
-		)
-		(property "Value" "+3V3"
-			(at 49.53 21.59 0)
-			(effects
-				(font
-					(size 1.27 1.27)
-				)
-			)
-		)
-		(property "Footprint" ""
-			(at 49.53 26.67 0)
-			(effects
-				(font
-					(size 1.27 1.27)
-				)
-				(hide yes)
-			)
-		)
-		(property "Datasheet" ""
-			(at 49.53 26.67 0)
-			(effects
-				(font
-					(size 1.27 1.27)
-				)
-				(hide yes)
-			)
-		)
-		(property "Description" "Power symbol creates a global label with name \"+3V3\""
-			(at 49.53 26.67 0)
-			(effects
-				(font
-					(size 1.27 1.27)
-				)
-				(hide yes)
-			)
-		)
-		(pin "1"
-		)
-		(instances
-			(project "erc_demo"
-				(path "/c0ee82df-0125-4137-95bd-a880c945d7bb"
-					(reference "#PWR1")
-					(unit 1)
-				)
-			)
-		)
-	)
-	(symbol
 		(lib_id "Device:R")
 		(at 53.34 53.34 0)
@@
 		(on_board yes)
 		(dnp no)
-		(property "Reference" "R4"
+		(property "Reference" "R11"
 			(at 52.07 49.53 0)
 			(effects
@@
 		)
 		(instances
+			(project "prj_erc"
+				(path "/4193f6fe-8549-4492-bb81-b789debaebf4/25c39909-a44f-4c3e-9fa4-3d0496d358a5"
+					(reference "R11")
+					(unit 1)
+				)
+			)
 			(project "erc_demo2"
 				(path "/c0ee82df-0125-4137-95bd-a880c945d7bb"
@@
 		(on_board yes)
 		(dnp no)
-		(property "Reference" "R8"
+		(property "Reference" "R15"
 			(at 62.23 49.53 0)
 			(effects
@@
 		)
 		(instances
+			(project "prj_erc"
+				(path "/4193f6fe-8549-4492-bb81-b789debaebf4/25c39909-a44f-4c3e-9fa4-3d0496d358a5"
+					(reference "R15")
+					(unit 1)
+				)
+			)
 			(project "erc_demo2"
 				(path "/c0ee82df-0125-4137-95bd-a880c945d7bb"
@@
 		(on_board yes)
 		(dnp no)
-		(property "Reference" "#FLG2"
+		(property "Reference" "#FLG0103"
 			(at 44.45 31.115 0)
 			(effects
@@
 		)
 		(instances
+			(project "prj_erc"
+				(path "/4193f6fe-8549-4492-bb81-b789debaebf4/25c39909-a44f-4c3e-9fa4-3d0496d358a5"
+					(reference "#FLG0103")
+					(unit 1)
+				)
+			)
 			(project "erc_demo"
 				(path "/c0ee82df-0125-4137-95bd-a880c945d7bb"
@@
 		(on_board yes)
 		(dnp no)
-		(property "Reference" "R7"
+		(property "Reference" "R16"
 			(at 62.23 68.58 0)
 			(effects
@@
 		)
 		(instances
+			(project "prj_erc"
+				(path "/4193f6fe-8549-4492-bb81-b789debaebf4/25c39909-a44f-4c3e-9fa4-3d0496d358a5"
+					(reference "R16")
+					(unit 1)
+				)
+			)
 			(project "erc_demo2"
 				(path "/c0ee82df-0125-4137-95bd-a880c945d7bb"
@@
 		(on_board yes)
 		(dnp no)
-		(property "Reference" "J5"
+		(property "Reference" "J4"
 			(at 13.208 64.77 0)
 			(effects
@@
 		)
 		(instances
+			(project "prj_erc"
+				(path "/4193f6fe-8549-4492-bb81-b789debaebf4/25c39909-a44f-4c3e-9fa4-3d0496d358a5"
+					(reference "J4")
+					(unit 1)
+				)
+			)
 			(project "erc_demo2"
 				(path "/c0ee82df-0125-4137-95bd-a880c945d7bb"
@@
 		(on_board yes)
 		(dnp no)
-		(property "Reference" "R2"
+		(property "Reference" "R9"
 			(at 46.99 49.53 0)
 			(effects
@@
 		)
 		(instances
+			(project "prj_erc"
+				(path "/4193f6fe-8549-4492-bb81-b789debaebf4/25c39909-a44f-4c3e-9fa4-3d0496d358a5"
+					(reference "R9")
+					(unit 1)
+				)
+			)
 			(project "erc_demo"
 				(path "/c0ee82df-0125-4137-95bd-a880c945d7bb"
@@
 		(on_board yes)
 		(dnp no)
-		(property "Reference" "R1"
+		(property "Reference" "R10"
 			(at 46.99 68.58 0)
 			(effects
@@
 		)
 		(instances
+			(project "prj_erc"
+				(path "/4193f6fe-8549-4492-bb81-b789debaebf4/25c39909-a44f-4c3e-9fa4-3d0496d358a5"
+					(reference "R10")
+					(unit 1)
+				)
+			)
 			(project ""
 				(path "/c0ee82df-0125-4137-95bd-a880c945d7bb"
@@
 		(on_board yes)
 		(dnp no)
-		(property "Reference" "R6"
+		(property "Reference" "R13"
 			(at 57.15 49.53 0)
 			(effects
@@
 		)
 		(instances
+			(project "prj_erc"
+				(path "/4193f6fe-8549-4492-bb81-b789debaebf4/25c39909-a44f-4c3e-9fa4-3d0496d358a5"
+					(reference "R13")
+					(unit 1)
+				)
+			)
 			(project "erc_demo2"
 				(path "/c0ee82df-0125-4137-95bd-a880c945d7bb"
@@
 		(on_board yes)
 		(dnp no)
-		(property "Reference" "R3"
+		(property "Reference" "R12"
 			(at 52.07 68.58 0)
 			(effects
@@
 		)
 		(instances
+			(project "prj_erc"
+				(path "/4193f6fe-8549-4492-bb81-b789debaebf4/25c39909-a44f-4c3e-9fa4-3d0496d358a5"
+					(reference "R12")
+					(unit 1)
+				)
+			)
 			(project "erc_demo2"
 				(path "/c0ee82df-0125-4137-95bd-a880c945d7bb"
@@
 		(dnp no)
 		(fields_autoplaced yes)
-		(property "Reference" "J4"
+		(property "Reference" "J6"
 			(at 73.66 62.2299 0)
 			(effects
@@
 		)
 		(instances
+			(project "prj_erc"
+				(path "/4193f6fe-8549-4492-bb81-b789debaebf4/25c39909-a44f-4c3e-9fa4-3d0496d358a5"
+					(reference "J6")
+					(unit 1)
+				)
+			)
 			(project ""
 				(path "/c0ee82df-0125-4137-95bd-a880c945d7bb"
@@
 		(dnp no)
 		(fields_autoplaced yes)
-		(property "Reference" "#PWR3"
+		(property "Reference" "#PWR0108"
 			(at 48.26 83.82 0)
 			(effects
@@
 		)
 		(instances
+			(project "prj_erc"
+				(path "/4193f6fe-8549-4492-bb81-b789debaebf4/25c39909-a44f-4c3e-9fa4-3d0496d358a5"
+					(reference "#PWR0108")
+					(unit 1)
+				)
+			)
 			(project "erc_demo"
 				(path "/c0ee82df-0125-4137-95bd-a880c945d7bb"
@@
 		(dnp no)
 		(fields_autoplaced yes)
-		(property "Reference" "#PWR4"
+		(property "Reference" "#PWR0105"
 			(at 48.26 49.53 0)
 			(effects
@@
 		)
 		(instances
+			(project "prj_erc"
+				(path "/4193f6fe-8549-4492-bb81-b789debaebf4/25c39909-a44f-4c3e-9fa4-3d0496d358a5"
+					(reference "#PWR0105")
+					(unit 1)
+				)
+			)
 			(project "erc_demo"
 				(path "/c0ee82df-0125-4137-95bd-a880c945d7bb"
@@
 		(on_board yes)
 		(dnp no)
-		(property "Reference" "J3"
+		(property "Reference" "J5"
 			(at 34.29 24.13 0)
 			(effects
@@
 		)
 		(instances
+			(project "prj_erc"
+				(path "/4193f6fe-8549-4492-bb81-b789debaebf4/25c39909-a44f-4c3e-9fa4-3d0496d358a5"
+					(reference "J5")
+					(unit 1)
+				)
+			)
 			(project ""
 				(path "/c0ee82df-0125-4137-95bd-a880c945d7bb"
 					(reference "J3")
-					(unit 1)
-				)
-			)
-		)
-	)
-	(symbol
-		(lib_id "power:GND")
-		(at 49.53 29.21 0)
-		(unit 1)
-		(exclude_from_sim no)
-		(in_bom yes)
-		(on_board yes)
-		(dnp no)
-		(fields_autoplaced yes)
-		(property "Reference" "#PWR2"
-			(at 49.53 35.56 0)
-			(effects
-				(font
-					(size 1.27 1.27)
-				)
-				(hide yes)
-			)
-		)
-		(property "Value" "GND"
-			(at 49.53 34.29 0)
-			(effects
-				(font
-					(size 1.27 1.27)
-				)
-			)
-		)
-		(property "Footprint" ""
-			(at 49.53 29.21 0)
-			(effects
-				(font
-					(size 1.27 1.27)
-				)
-				(hide yes)
-			)
-		)
-		(property "Datasheet" ""
-			(at 49.53 29.21 0)
-			(effects
-				(font
-					(size 1.27 1.27)
-				)
-				(hide yes)
-			)
-		)
-		(property "Description" "Power symbol creates a global label with name \"GND\" , ground"
-			(at 49.53 29.21 0)
-			(effects
-				(font
-					(size 1.27 1.27)
-				)
-				(hide yes)
-			)
-		)
-		(pin "1"
-		)
-		(instances
-			(project "erc_demo"
-				(path "/c0ee82df-0125-4137-95bd-a880c945d7bb"
-					(reference "#PWR2")
 					(unit 1)
 				)
@@
 		(on_board yes)
 		(dnp no)
-		(property "Reference" "R5"
+		(property "Reference" "R14"
 			(at 57.15 68.58 0)
 			(effects
@@
 		)
 		(instances
+			(project "prj_erc"
+				(path "/4193f6fe-8549-4492-bb81-b789debaebf4/25c39909-a44f-4c3e-9fa4-3d0496d358a5"
+					(reference "R14")
+					(unit 1)
+				)
+			)
 			(project "erc_demo2"
 				(path "/c0ee82df-0125-4137-95bd-a880c945d7bb"
@@
 		(on_board yes)
 		(dnp no)
-		(property "Reference" "#FLG1"
+		(property "Reference" "#FLG0104"
 			(at 44.45 24.765 0)
 			(effects
@@
 		)
 		(instances
+			(project "prj_erc"
+				(path "/4193f6fe-8549-4492-bb81-b789debaebf4/25c39909-a44f-4c3e-9fa4-3d0496d358a5"
+					(reference "#FLG0104")
+					(unit 1)
+				)
+			)
 			(project ""
 				(path "/c0ee82df-0125-4137-95bd-a880c945d7bb"
